Commit message: Adding phone and vive tracker teleoperation

File: assets/g1/g1_inspire_gen4.urdf (robot description, URDF)
Before this commit: robot g1_inspire_gen4, 73 links, 72 joints
Joints:
- joint left_index_2_joint: limit lower=0. upper=1.5999998 effort=3.5 velocity=17453.2925199 -> lower=0. upper=1.5999998 effort=3.5 velocity=10.0; mimic (none) -> joint=left_index_1_joint multiplier=1.05 offset=0.
- joint left_little_2_joint: limit lower=0. upper=1.5999998 effort=3.5 velocity=17453.2925199 -> lower=0. upper=1.5999998 effort=3.5 velocity=10.0; mimic (none) -> joint=left_little_1_joint multiplier=1.05 offset=0.
- joint left_middle_2_joint: limit lower=0. upper=1.5999998 effort=3.5 velocity=17453.2925199 -> lower=0. upper=1.5999998 effort=3.5 velocity=10.0; mimic (none) -> joint=left_middle_1_joint multiplier=1.05 offset=0.
- joint left_ring_2_joint: limit lower=0. upper=1.5999998 effort=3.5 velocity=17453.2925199 -> lower=0. upper=1.5999998 effort=3.5 velocity=10.0; mimic (none) -> joint=left_ring_1_joint multiplier=1.05 offset=0.
- joint left_thumb_2_joint: limit lower=-0.95 upper=0. effort=5. velocity=17453.2925199 -> lower=-0.95 upper=0. effort=5. velocity=10.0
- joint left_thumb_3_joint: limit lower=-0.3799999 upper=0. effort=5. velocity=17453.2925199 -> lower=-0.3799999 upper=0. effort=5. velocity=10.0; mimic (none) -> joint=left_thumb_2_joint multiplier=0.4 offset=0.
- joint left_thumb_4_joint: limit lower=-0.5699999 upper=0. effort=5. velocity=17453.2925199 -> lower=-0.5699999 upper=0. effort=5. velocity=10.0; mimic (none) -> joint=left_thumb_2_joint multiplier=0.6 offset=0.
- joint right_index_1_joint: limit lower=0. upper=1.5238094 effort=10000000. velocity=17453.2925199 -> lower=0. upper=1.5238094 effort=10000000. velocity=10.0
- joint right_index_2_joint: limit lower=0. upper=1.5999998 effort=3.5 velocity=17453.2925199 -> lower=0. upper=1.5999998 effort=3.5 velocity=10.0; mimic (none) -> joint=right_index_1_joint multiplier=1.05 offset=0.
- joint right_little_1_joint: limit lower=0. upper=1.5238094 effort=10000000. velocity=17453.2925199 -> lower=0. upper=1.5238094 effort=10000000. velocity=10.0
- joint right_little_2_joint: limit lower=0. upper=1.5999998 effort=3.5 velocity=17453.2925199 -> lower=0. upper=1.5999998 effort=3.5 velocity=10.0; mimic (none) -> joint=right_little_1_joint multiplier=1.05 offset=0.
- joint right_middle_1_joint: limit lower=0. upper=1.5238094 effort=10000000. velocity=17453.2925199 -> lower=0. upper=1.5238094 effort=10000000. velocity=10.0
- joint right_middle_2_joint: limit lower=0. upper=1.5999998 effort=3.5 velocity=17453.2925199 -> lower=0. upper=1.5999998 effort=3.5 velocity=10.0; mimic (none) -> joint=right_middle_1_joint multiplier=1.05 offset=0.
- joint right_ring_1_joint: limit lower=0. upper=1.5238094 effort=10000000. velocity=17453.2925199 -> lower=0. upper=1.5238094 effort=10000000. velocity=10.0
- joint right_ring_2_joint: limit lower=0. upper=1.5999998 effort=3.5 velocity=17453.2925199 -> lower=0. upper=1.5999998 effort=3.5 velocity=10.0; mimic (none) -> joint=right_ring_1_joint multiplier=1.05 offset=0.
- joint right_thumb_1_joint: limit lower=0. upper=1.7 effort=10000000. velocity=17453.2925199 -> lower=0. upper=1.7 effort=10000000. velocity=10.0
- joint right_thumb_2_joint: limit lower=0. upper=0.95 effort=10000000. velocity=17453.2925199 -> lower=0. upper=0.95 effort=10000000. velocity=10.0
- joint right_thumb_3_joint: limit lower=0. upper=0.38 effort=5. velocity=17453.2925199 -> lower=0. upper=0.38 effort=5. velocity=10.0; mimic (none) -> joint=right_thumb_2_joint multiplier=0.4 offset=0.
- joint right_thumb_4_joint: limit lower=0. upper=0.57 effort=5. velocity=17453.2925199 -> lower=0. upper=0.57 effort=5. velocity=10.0; mimic (none) -> joint=right_thumb_2_joint multiplier=0.6 offset=0.
