Commit message: dding edits before iros

File: assets/g1/g1_body29_hand14.urdf (robot description, URDF)
Before this commit: robot g1, 53 links, 52 joints
Joints:
- joint left_shoulder_roll_joint: limit lower=-1.5882 upper=2.2515 effort=25 velocity=37 -> lower=-0.05 upper=2.2515 effort=25 velocity=37
- joint right_shoulder_roll_joint: limit lower=-2.2515 upper=1.5882 effort=25 velocity=37 -> lower=-2.2515 upper=0.05 effort=25 velocity=37

File: assets/g1/g1_inspire_gen4.urdf (robot description, URDF)
Before this commit: robot g1_inspire_gen4, 73 links, 72 joints
Joints:
- joint left_shoulder_roll_joint: limit lower=-1.5882 upper=2.2515 effort=25 velocity=37 -> lower=-0.05 upper=2.2515 effort=25 velocity=37
- joint right_shoulder_roll_joint: limit lower=-2.2515 upper=1.5882 effort=25 velocity=37 -> lower=-2.2515 upper=0.05 effort=25 velocity=37
